File: hardware/downlink_board/downlink_board.kicad_pcb (KiCad board)
At the start: 2 copper layers, 65 x 56 mm, 55 parts, among them J1 USB_C_Receptacle_USB2.0, J2 SCREEN, J3 GPIO, J4 PROGRAM, SW1 RPi_{ON}, SW2 RPi_{OFF}, SW3 MCU_{RST}, U1 AZ1117-3.3, U2 TPS563208DDCR, U3 STM32F103C8Tx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

Commit message: BOM adjustments
Parts:
- R15: value 50k -> 54k9
Changed lines of the file:
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@@
         (effects (font (size 1 1) (thickness 0.15)))
     )
-    (fp_text value "50k" (at 0.1125 1.43) (layer "F.Fab")
+    (fp_text value "54k9" (at 0.1125 1.43) (layer "F.Fab")
         (effects (font (size 1 1) (thickness 0.15)))
     )
@@
     (pad "" np_thru_hole circle (at 8.8 26.4 90) (size 4.9 4.9) (drill 4.9) (layers "*.Cu" "*.Mask"))
     (pad "" np_thru_hole circle (at 8.8 52.8 90) (size 4.9 4.9) (drill 4.9) (layers "*.Cu" "*.Mask"))
-    (pad "1" thru_hole roundrect (at 0 0 90) (size 4.4 4.4) (drill 3) (layers "*.Cu" "*.Mask") (roundrect_rratio 0.056818)
+    (pad "1" thru_hole roundrect (at 0 0 90) (size 4.4 4.4) (drill 3) (layers "*.Cu" "*.Mask") (roundrect_rratio 0.05681795455)
       (net 7 "+BATT") (pinfunction "+") (pintype "passive"))
     (pad "2" thru_hole circle (at 8.8 0 90) (size 4.4 4.4) (drill 3) (layers "*.Cu" "*.Mask")
@@
     (fp_line (start 10 3.2) (end 10 -3.2)
       (stroke (width 0.1) (type solid)) (layer "F.Fab"))
-    (pad "1" thru_hole roundrect (at 0 0 180) (size 1.7 1.95) (drill 0.95) (layers "*.Cu" "*.Mask") (roundrect_rratio 0.147059)
+    (pad "1" thru_hole roundrect (at 0 0 180) (size 1.7 1.95) (drill 0.95) (layers "*.Cu" "*.Mask") (roundrect_rratio 0.1470588235)
       (net 1 "GND") (pinfunction "Pin_1") (pintype "passive"))
     (pad "2" thru_hole oval (at 2.5 0 180) (size 1.7 1.95) (drill 0.95) (layers "*.Cu" "*.Mask")
