File: hardware/downlink_board/downlink_board.kicad_sch (KiCad schematic)
At the start: 51 parts, among them J2 SCREEN, J2 USB_C_Receptacle_USB2.0, J3 GPIO, J4 PROGRAM, SW1 MCU_{RST}, SW1 RPi_{ON}, SW2 RPi_{OFF}, U1 nRF24L01, U2 STM32F103C8Tx, U2 TPS563208DDCR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

Commit message: BOM adjustments
Parts:
- R18: value 50k -> 54k9
Changed lines of the file:
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@@
       (effects (font (size 1.27 1.27)))
     )
-    (property "Value" "50k" (at 130.81 69.85 0)
+    (property "Value" "54k9" (at 130.81 69.85 0)
       (effects (font (size 1.27 1.27)))
     )
